File: ESP.sch (KiCad schematic (older format))
At the start: 24 parts, among them P1 CONN, P2 CONN, P3 CONN, P4 CONN, P5 CONN, U1 4N35, U2 ESP-13-WROOM-02, U3 MOC3041M, U4 BT808

Commit message: PCB Wiring
Parts:
- added P6: RX TX G, Pin_Headers:Pin_Header_Straight_1x03, symbol CONN_01X03
- P1: value CONN -> BTN
- P2: value CONN -> - +
- P3: value CONN -> PROG
- P4: value CONN -> LAMP
Connections:
- net GND: now also P6.1 (P1)
- net at U2.11 (RXD): now also P6.3 (P3)
- net at U2.12 (TXD): now also P6.2 (P2)
Changed lines of the file:
@@
 LIBS:contrib
 LIBS:valves
-LIBS:ESP8266
 LIBS:ESP-cache
 EELAYER 25 0
@@
 F 0 "U1" H 2300 4400 50  0000 L CNN
 F 1 "4N35" H 2500 4400 50  0000 L CNN
-F 2 "Sockets_DIP:DIP-6__300_ELL" H 2300 4000 50  0000 L CIN
+F 2 "Sockets_DIP:DIP-6__300_ELL" H 2300 4000 50  0001 L CIN
 F 3 "" H 2500 4200 50  0000 L CNN
 	1    2500 4200
@@
 F 0 "U3" H 6540 4890 50  0000 L CNN
 F 1 "MOC3041M" H 6750 4900 50  0000 L CNN
-F 2 "Sockets_DIP:DIP-6__300_ELL" H 6550 4500 50  0000 L CIN
+F 2 "Sockets_DIP:DIP-6__300_ELL" H 6550 4500 50  0001 L CIN
 F 3 "" H 6725 4700 50  0000 L CNN
 	1    6750 4700
@@
 P 1200 4150
 F 0 "P1" H 1200 4300 50  0000 C CNN
-F 1 "CONN" V 1300 4150 50  0000 C CNN
-F 2 "Connect:bornier2" H 1200 4150 60  0000 C CNN
+F 1 "BTN" V 1300 4150 50  0000 C CNN
+F 2 "Connect:bornier2" H 1200 4150 60  0001 C CNN
 F 3 "" H 1200 4150 60  0000 C CNN
 	1    1200 4150
@@
 P 9900 4850
 F 0 "P4" H 9900 5000 50  0000 C CNN
-F 1 "CONN" V 10000 4850 50  0000 C CNN
-F 2 "Connect:bornier2" H 9900 4850 60  0000 C CNN
+F 1 "LAMP" V 10000 4850 50  0000 C CNN
+F 2 "Connect:bornier2" H 9900 4850 60  0001 C CNN
 F 3 "" H 9900 4850 60  0000 C CNN
 	1    9900 4850
@@
 F 0 "C1" H 8775 5100 50  0000 L CNN
 F 1 "0.1 400V" H 8775 4900 50  0000 L CNN
-F 2 "Capacitors_ThroughHole:C_Rect_L18_W7_P15" H 8788 4850 30  0000 C CNN
+F 2 "Capacitors_ThroughHole:C_Rect_L18_W7_P15" H 8788 4850 30  0001 C CNN
 F 3 "" H 8750 5000 60  0000 C CNN
 	1    8750 5000
@@
 F 0 "R12" V 8830 4550 50  0000 C CNN
 F 1 "100" V 8750 4550 50  0000 C CNN
-F 2 "Resistors_ThroughHole:Resistor_Horizontal_RM15mm" V 8680 4550 30  0000 C CNN
+F 2 "Resistors_ThroughHole:Resistor_Horizontal_RM15mm" V 8680 4550 30  0001 C CNN
 F 3 "" H 8750 4550 30  0000 C CNN
 	1    8750 4550
@@
 F 0 "U4" H 7750 5150 50  0000 C CNN
 F 1 "BT808" H 7700 4550 50  0000 C CNN
-F 2 "Transistors_TO-220:TO-220_Neutral123_Vertical_LargePads" H 8000 4800 60  0000 C CNN
+F 2 "Transistors_TO-220:TO-220_Neutral123_Vertical_LargePads" H 8000 4800 60  0001 C CNN
 F 3 "" H 8000 4800 60  0000 C CNN
 	1    8000 4800
@@
 F 0 "R1" V 1930 4100 50  0000 C CNN
 F 1 "1K" V 1850 4100 50  0000 C CNN
-F 2 "Resistors_ThroughHole:Resistor_Horizontal_RM10mm" V 1780 4100 30  0000 C CNN
+F 2 "Resistors_ThroughHole:Resistor_Horizontal_RM10mm" V 1780 4100 30  0001 C CNN
 F 3 "" H 1850 4100 30  0000 C CNN
 	1    1850 4100
@@
 F 0 "R11" V 7630 5150 50  0000 C CNN
 F 1 "470" V 7550 5150 50  0000 C CNN
-F 2 "Resistors_ThroughHole:Resistor_Horizontal_RM10mm" V 7480 5150 30  0000 C CNN
+F 2 "Resistors_ThroughHole:Resistor_Horizontal_RM10mm" V 7480 5150 30  0001 C CNN
 F 3 "" H 7550 5150 30  0000 C CNN
 	1    7550 5150
@@
 F 0 "R10" V 7630 4400 50  0000 C CNN
 F 1 "390" V 7550 4400 50  0000 C CNN
-F 2 "Resistors_ThroughHole:Resistor_Horizontal_RM10mm" V 7480 4400 30  0000 C CNN
+F 2 "Resistors_ThroughHole:Resistor_Horizontal_RM10mm" V 7480 4400 30  0001 C CNN
 F 3 "" H 7550 4400 30  0000 C CNN
 	1    7550 4400
@@
 F 0 "F1" H 9500 4850 50  0000 C CNN
 F 1 "FUSE" H 9300 4750 50  0000 C CNN
-F 2 "Fuse_Holders_and_Fuses:Fuseholder5x20_horiz_SemiClosed_Casing10x25mm" H 9400 4800 60  0000 C CNN
+F 2 "Fuse_Holders_and_Fuses:Fuseholder5x20_horiz_SemiClosed_Casing10x25mm" H 9400 4800 60  0001 C CNN
 F 3 "" H 9400 4800 60  0000 C CNN
 	1    9400 4800
@@
 F 0 "R9" V 6330 4600 50  0000 C CNN
 F 1 "68" V 6250 4600 50  0000 C CNN
-F 2 "Resistors_ThroughHole:Resistor_Horizontal_RM10mm" V 6180 4600 30  0000 C CNN
+F 2 "Resistors_ThroughHole:Resistor_Horizontal_RM10mm" V 6180 4600 30  0001 C CNN
 F 3 "" H 6250 4600 30  0000 C CNN
 	1    6250 4600
@@
 F 0 "R8" V 6080 4750 50  0000 C CNN
 F 1 "100" V 6000 4750 50  0000 C CNN
-F 2 "Resistors_ThroughHole:Resistor_Horizontal_RM10mm" V 5930 4750 30  0000 C CNN
+F 2 "Resistors_ThroughHole:Resistor_Horizontal_RM10mm" V 5930 4750 30  0001 C CNN
 F 3 "" H 6000 4750 30  0000 C CNN
 	1    6000 4750
@@
 F 0 "D1" H 6000 5250 50  0000 C CNN
 F 1 "LED" H 6000 5050 50  0000 C CNN
-F 2 "LEDs:LED-3MM" H 6000 5150 60  0000 C CNN
+F 2 "LEDs:LED-3MM" H 6000 5150 60  0001 C CNN
 F 3 "" H 6000 5150 60  0000 C CNN
 	1    6000 5150
@@
 F 0 "R3" V 3280 4100 50  0000 C CNN
 F 1 "10K" V 3200 4100 50  0000 C CNN
-F 2 "Resistors_ThroughHole:Resistor_Horizontal_RM10mm" V 3130 4100 30  0000 C CNN
+F 2 "Resistors_ThroughHole:Resistor_Horizontal_RM10mm" V 3130 4100 30  0001 C CNN
 F 3 "" H 3200 4100 30  0000 C CNN
 	1    3200 4100
@@
 P 1200 4750
 F 0 "P2" H 1200 4900 50  0000 C CNN
-F 1 "CONN" V 1300 4750 50  0000 C CNN
-F 2 "Connect:bornier2" H 1200 4750 60  0000 C CNN
+F 1 "- +" V 1300 4750 50  0000 C CNN
+F 2 "Connect:bornier2" H 1200 4750 60  0001 C CNN
 F 3 "" H 1200 4750 60  0000 C CNN
 	1    1200 4750
@@
 F 0 "U2" H 5050 1400 50  0000 C CNN
 F 1 "ESP-13-WROOM-02" H 5050 1950 50  0000 C CNN
-F 2 "ESP8266:ESP-13-WROOM-02" H 4950 1500 50  0000 C CNN
+F 2 "ESP8266:ESP-13-WROOM-02" H 4950 1500 50  0001 C CNN
 F 3 "" H 4950 1500 50  0001 C CNN
 	1    5050 1500
@@
 F 0 "R6" V 3730 1000 50  0000 C CNN
 F 1 "1K" V 3650 1000 50  0000 C CNN
-F 2 "Resistors_ThroughHole:Resistor_Horizontal_RM10mm" V 3580 1000 30  0000 C CNN
+F 2 "Resistors_ThroughHole:Resistor_Horizontal_RM10mm" V 3580 1000 30  0001 C CNN
 F 3 "" H 3650 1000 30  0000 C CNN
 	1    3650 1000
@@
 F 0 "R5" V 3580 1000 50  0000 C CNN
 F 1 "1K" V 3500 1000 50  0000 C CNN
-F 2 "Resistors_ThroughHole:Resistor_Horizontal_RM10mm" V 3430 1000 30  0000 C CNN
+F 2 "Resistors_ThroughHole:Resistor_Horizontal_RM10mm" V 3430 1000 30  0001 C CNN
 F 3 "" H 3500 1000 30  0000 C CNN
 	1    3500 1000
@@
 F 0 "R4" V 3430 1000 50  0000 C CNN
 F 1 "1K" V 3350 1000 50  0000 C CNN
-F 2 "Resistors_ThroughHole:Resistor_Horizontal_RM10mm" V 3280 1000 30  0000 C CNN
+F 2 "Resistors_ThroughHole:Resistor_Horizontal_RM10mm" V 3280 1000 30  0001 C CNN
 F 3 "" H 3350 1000 30  0000 C CNN
 	1    3350 1000
@@
 F 0 "R2" V 3280 1000 50  0000 C CNN
 F 1 "1K" V 3200 1000 50  0000 C CNN
-F 2 "Resistors_ThroughHole:Resistor_Horizontal_RM10mm" V 3130 1000 30  0000 C CNN
+F 2 "Resistors_ThroughHole:Resistor_Horizontal_RM10mm" V 3130 1000 30  0001 C CNN
 F 3 "" H 3200 1000 30  0000 C CNN
 	1    3200 1000
@@
 F 0 "R7" V 3730 2100 50  0000 C CNN
 F 1 "1K" V 3650 2100 50  0000 C CNN
-F 2 "Resistors_ThroughHole:Resistor_Horizontal_RM10mm" V 3580 2100 30  0000 C CNN
+F 2 "Resistors_ThroughHole:Resistor_Horizontal_RM10mm" V 3580 2100 30  0001 C CNN
 F 3 "" H 3650 2100 30  0000 C CNN
 	1    3650 2100
@@
 P 3150 2050
 F 0 "P3" H 3150 2200 50  0000 C CNN
-F 1 "CONN" V 3250 2050 50  0000 C CNN
-F 2 "Pin_Headers:Pin_Header_Straight_1x02" H 3150 2050 60  0000 C CNN
+F 1 "PROG" V 3250 2050 50  0000 C CNN
+F 2 "Pin_Headers:Pin_Header_Straight_1x02" H 3150 2050 60  0001 C CNN
 F 3 "" H 3150 2050 60  0000 C CNN
 	1    3150 2050
@@
 F 0 "P5" H 1700 1500 50  0000 C CNN
 F 1 "CONN" V 1800 1350 50  0000 C CNN
-F 2 "Connect:bornier2" H 1700 1350 60  0000 C CNN
+F 2 "Connect:bornier2" H 1700 1350 60  0001 C CNN
 F 3 "" H 1700 1350 60  0000 C CNN
 	1    1700 1350
@@
 	3350 2300 6150 2300
 Wire Wire Line
-	6150 2300 6150 1200
-Wire Wire Line
-	6000 1700 6150 1700
-Wire Wire Line
 	3950 2000 3950 2400
 Wire Wire Line
@@
 	1400 4800 2100 4800
 Wire Wire Line
-	1400 4700 1650 4700
+	1650 4700 1400 4700
 Connection ~ 3000 4200
 Wire Wire Line
@@
 Wire Wire Line
 	8750 4850 8750 4700
+$Comp
+L CONN_01X03 P6
+U 1 1 561C43DA
+P 7250 1800
+F 0 "P6" H 7250 2000 50  0000 C CNN
+F 1 "RX TX G" V 7350 1800 50  0000 C CNN
+F 2 "Pin_Headers:Pin_Header_Straight_1x03" H 7250 1800 60  0001 C CNN
+F 3 "" H 7250 1800 60  0000 C CNN
+	1    7250 1800
+	1    0    0    -1
+$EndComp
+Wire Wire Line
+	7050 1900 6000 1900
+Wire Wire Line
+	6000 1800 7050 1800
+Wire Wire Line
+	6150 2300 6150 1200
+Wire Wire Line
+	6000 1700 7050 1700
 $EndSCHEMATC
