File: ESP.kicad_pcb (KiCad board)
At the start: 2 copper layers, 24 parts, among them P1 CONN, P2 CONN, P3 CONN, P4 CONN, P5 CONN, U1 4N35, U2 ESP-13-WROOM-02, U3 MOC3041M, U4 BT808

Commit message: PCB redistribution
Parts:
- moved R5 31.1 mm to (129.5, 84.5), turned to 90 degrees
- moved R4 27.5 mm to (126.0, 84.5), turned to 90 degrees
- moved R2 24.3 mm to (122.5, 84.5), turned to 90 degrees
- moved R7 21.8 mm to (119.0, 84.5), turned to 270 degrees
- moved R1 21.6 mm to (101.5, 85.0)
- moved P3 20.5 mm to (109.5, 77.0), turned to 180 degrees
- moved R6 20.2 mm to (115.5, 84.5), turned to 90 degrees
- moved R3 20.2 mm to (99.8, 67.0)
- moved U1 20.1 mm to (99.8, 75.5)
- moved P1 19.3 mm to (88.2, 75.2)
- moved P2 19.3 mm to (88.2, 86.8)
- moved P5 19.3 mm to (88.2, 63.2)
- moved R8 14.3 mm to (136.0, 70.8), turned to 90 degrees
- moved D1 12.9 mm to (136.0, 58.8)
- moved U2 12.4 mm to (113.5, 64.2)
Routing:
- net BUTTONS: track 67.8 -> 0.00 mm
- net +3V3: track 66.3 -> 15.5 mm
- net Net-(P3-Pad2): track 31.4 -> 4.45 mm
- net Net-(R1-Pad1): track 18.5 -> 0.00 mm
- net Net-(P1-Pad2): track 18.0 -> 0.00 mm
- net Net-(P2-Pad1): track 17.8 -> 0.00 mm
- net Net-(D1-Pad2): track 20.1 -> 4.38 mm
- net Net-(R7-Pad1): track 9.83 -> 0.00 mm
- net Net-(R6-Pad2): track 7.92 -> 0.00 mm
- net Net-(R2-Pad2): track 7.83 -> 0.58 mm
- net Net-(R5-Pad2): track 34.2 -> 27.2 mm, vias 2 -> 0
- net Net-(P1-Pad1): track 6.42 -> 0.00 mm
- net GND: track 132.8 -> 126.9 mm
- net Net-(F1-Pad1): track 32.0 -> 35.8 mm
- net MAINS: track 10.5 -> 12.0 mm
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
Commit message: PCB Wiring
Parts:
- added P6: RX TX G, Pin_Headers:Pin_Header_Straight_1x03, F.Cu at (103.8, 86.5)
- P1: value CONN -> BTN
- P2: value CONN -> - +
- P3: value CONN -> PROG
- P4: value CONN -> LAMP
- moved R1 25.7 mm to (105.0, 59.5)
- moved U1 7.25 mm to (105.0, 70.5), turned to 180 degrees
- moved R4 7.00 mm to (119.0, 84.5)
- moved R7 7.00 mm to (126.0, 84.5)
- moved P3 6.73 mm to (103.8, 80.5), turned to 90 degrees
- moved R3 6.60 mm to (105.0, 63.0)
- moved P1 4.07 mm to (92.2, 74.5)
- moved P5 4.07 mm to (92.2, 62.5)
- moved P2 4.01 mm to (92.2, 86.5)
Connections:
- U2 pad 11: (no net) -> Net-(P6-Pad3)
- U2 pad 12: (no net) -> Net-(P6-Pad2)
Routing:
- net BUTTONS: track 0.00 -> 72.2 mm, vias 0 -> 2
- net +3V3: track 15.5 -> 77.2 mm, vias 0 -> 2
- net Net-(P2-Pad1): track 0.00 -> 48.2 mm
- net Net-(P6-Pad2): track 0.00 -> 40.9 mm
- net Net-(P6-Pad3): track 0.00 -> 33.9 mm
- net GND: track 126.9 -> 154.8 mm, vias 0 -> 2
- net Net-(P1-Pad2): track 0.00 -> 23.5 mm
- net Net-(R6-Pad2): track 0.00 -> 19.6 mm, vias 0 -> 2
- net Net-(R7-Pad1): track 0.00 -> 19.2 mm, vias 0 -> 2
- net Net-(P3-Pad2): track 4.45 -> 19.8 mm, vias 0 -> 2
- net Net-(R2-Pad2): track 0.58 -> 15.1 mm, vias 0 -> 2
- net Net-(R5-Pad2): track 27.2 -> 18.8 mm, vias 0 -> 2
- net Net-(R1-Pad1): track 0.00 -> 8.24 mm
- net Net-(P1-Pad1): track 0.00 -> 6.92 mm
- net Net-(C1-Pad2): track 40.0 -> 40.5 mm

Commit message: PCB Edjes
Other:
- board outline added: 90.2 x 36.8 mm
Changed lines of the file:
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@@
     (links 44)
     (no_connects 0)
-    (area 0 0 0 0)
+    (area 86.309999 55.829999 176.580001 92.760001)
     (thickness 1.6)
-    (drawings 0)
+    (drawings 4)
     (tracks 218)
     (zones 0)
@@
     )
   )
+  (gr_line (start 86.36 92.71) (end 86.36 55.88) (angle 90) (layer Edge.Cuts) (width 0.1))
+  (gr_line (start 176.53 92.71) (end 86.36 92.71) (angle 90) (layer Edge.Cuts) (width 0.1))
+  (gr_line (start 176.53 55.88) (end 176.53 92.71) (angle 90) (layer Edge.Cuts) (width 0.1))
+  (gr_line (start 86.36 55.88) (end 176.53 55.88) (angle 90) (layer Edge.Cuts) (width 0.1))
   (segment (start 172 73) (end 164.5 73) (width 1) (layer F.Cu) (net 1))
   (segment (start 165.08 79.5) (end 172 79.5) (width 1) (layer F.Cu) (net 2))
@@
   (segment (start 105 72.25) (end 105 74.31) (width 0.25) (layer F.Cu) (net 11))
   (segment (start 99.92 67.17) (end 105 72.25) (width 0.25) (layer F.Cu) (net 11))
-  (segment (start 131.5 71.75) (end 133 71.75) (width 0.5) (layer F.Cu) (net 12) (status 400000))
-  (segment (start 133.75 65.5) (end 132.5 64.25) (width 0.5) (layer F.Cu) (net 12) (status 800000))
+  (segment (start 131.5 71.75) (end 133 71.75) (width 0.5) (layer F.Cu) (net 12))
+  (segment (start 133.75 65.5) (end 132.5 64.25) (width 0.5) (layer F.Cu) (net 12))
   (via (at 133.75 65.5) (size 0.6) (drill 0.4) (layers F.Cu B.Cu) (net 12))
   (segment (start 133.75 66.75) (end 133.75 65.5) (width 0.5) (layer B.Cu) (net 12))
@@
   (via (at 134 72.75) (size 0.6) (drill 0.4) (layers F.Cu B.Cu) (net 12))
   (segment (start 133 71.75) (end 134 72.75) (width 0.5) (layer F.Cu) (net 12))
-  (segment (start 132.5 64.25) (end 131.5 64.25) (width 0.5) (layer F.Cu) (net 12) (status C00000))
+  (segment (start 132.5 64.25) (end 131.5 64.25) (width 0.5) (layer F.Cu) (net 12))
   (segment (start 103.75 86.5) (end 103.75 85) (width 0.5) (layer F.Cu) (net 12))
   (segment (start 103.75 85) (end 105.25 83.5) (width 0.5) (layer F.Cu) (net 12))
